File: ikoka-stick-meshtastic-device.kicad_pcb (KiCad board)
At the start: 2 copper layers, 100 x 28 mm, 19 parts, among them J1 Conn_Coaxial, J2 Conn_01x07_Socket, J3 Conn_01x07_Socket, J4 Conn_01x02, J5 Conn_01x02, J6 Conn_01x04, Q1 AO3401A, SW1 SW_Push, U2 E22-900M30S, U3 XIAO-ESP32-S3-SMD

Commit message: feat: v3 - use E22P LoRa module (EN jumper JP1), ported from tahnok fork
E22P pin 6 is EN (must be high) instead of RXEN: route it to solder
jumper JP1 under the XIAO, bridged to 3V3 by default, D6 optional.
Pin 7 (T/R CTRL) stays on DIO2. Symbol and routing from
tahnok/ikoka-stick-meshtastic-device 366648b.

Co-Authored-By: Claude Opus 5.5 <noreply@anthropic.com>
Claude-Session: https://claude.ai/code/session_013aihWTyEvMfq2tmgNbS7qs
Parts:
- added JP1: SolderJumper_3_Bridged12, Jumper:SolderJumper-3_P1.3mm_Bridged12_RoundedPad1.0x1.5mm_NumberLabels, F.Cu at (213.7, 100.3)
- U2: value E22-900M30S -> E22P-915M30S
Connections:
- U2 pad 6: /LORA_RXEN -> Net-(JP1-C)
Routing:
- net Net-(JP1-C): track 0.00 -> 70.3 mm, vias 0 -> 2
- net /LORA_RXEN: track 66.3 -> 15.2 mm, vias 2 -> 1
- net +3V3: track 59.0 -> 68.3 mm
Other:
- board text added: "HW Ver.: 3.0.0"
- board text removed: "HW Ver.: 2.0.0"

Commit message: feat: v3 - swap OLED header J6 power pins (GND first), ported from tahnok fork
J6 pin 1 = GND, pin 2 = +3V3 as in tahnok 366648b; silk +/- marks.

Co-Authored-By: Claude Opus 5.5 <noreply@anthropic.com>
Claude-Session: https://claude.ai/code/session_013aihWTyEvMfq2tmgNbS7qs
Connections:
- J6 pad 1: +3V3 -> GND
- J6 pad 2: GND -> +3V3
Routing:
- net +3V3: track 68.3 -> 72.6 mm, vias 2 -> 4
Other:
- board text added: "+"
- board text added: "-"
Changed lines of the file:
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@@
 			(size 1.9 1)
 			(layers "F.Cu" "F.Mask" "F.Paste")
-			(net "+3V3")
+			(net "GND")
 			(pinfunction "Pin_1_1")
 			(pintype "passive")
@@
 			(size 1.9 1)
 			(layers "F.Cu" "F.Mask" "F.Paste")
-			(net "GND")
+			(net "+3V3")
 			(pinfunction "Pin_2_2")
 			(pintype "passive")
@@
 		)
 	)
+	(gr_text "+"
+		(at 169.5 98.35 0)
+		(layer "F.SilkS")
+		(effects
+			(font
+				(size 0.9 0.9)
+				(thickness 0.1)
+			)
+		)
+	)
+	(gr_text "-"
+		(at 177.5 95.5 180)
+		(layer "F.SilkS")
+		(effects
+			(font
+				(size 0.9 0.9)
+				(thickness 0.1)
+			)
+		)
+	)
 	(gr_text "JLCJLCJLCJLC"
 		(at 158 100 0)
@@
 	)
 	(via
+		(at 174.65 96.19)
+		(size 0.45)
+		(drill 0.3)
+		(layers "F.Cu" "B.Cu")
+		(net "GND")
+	)
+	(via
 		(at 187.25 106.425)
 		(size 0.45)
@@
 	)
 	(via
-		(at 171.35 98.73)
-		(size 0.45)
-		(drill 0.3)
-		(layers "F.Cu" "B.Cu")
-		(capping no)
-		(covering
-			(front no)
-			(back no)
-		)
-		(plugging
-			(front no)
-			(back no)
-		)
-		(filling no)
-		(net "GND")
-	)
-	(via
 		(at 166.64 88.425)
 		(size 0.45)
@@
 	)
 	(segment
-		(start 176.5 95.75)
-		(end 176.06 96.19)
-		(width 0.2)
-		(layer "F.Cu")
-		(net "+3V3")
-	)
-	(segment
 		(start 216.25 111)
 		(end 209.25 111)
@@
 	)
 	(segment
-		(start 176.06 96.19)
-		(end 174.65 96.19)
-		(width 0.2)
-		(layer "F.Cu")
-		(net "+3V3")
-	)
-	(segment
 		(start 208.166 103.416)
 		(end 200.5 95.75)
@@
 		(net "+3V3")
 	)
+	(via
+		(at 171.35 98.73)
+		(size 0.45)
+		(drill 0.3)
+		(layers "F.Cu" "B.Cu")
+		(net "+3V3")
+	)
+	(via
+		(at 176.5 95.75)
+		(size 0.45)
+		(drill 0.3)
+		(layers "F.Cu" "B.Cu")
+		(net "+3V3")
+	)
+	(segment
+		(start 176.5 95.75)
+		(end 173.52 98.73)
+		(width 0.2)
+		(layer "B.Cu")
+		(net "+3V3")
+	)
+	(segment
+		(start 173.52 98.73)
+		(end 171.35 98.73)
+		(width 0.2)
+		(layer "B.Cu")
+		(net "+3V3")
+	)
 	(segment
 		(start 194.5 99.175)
@@
 		(layer "F.Cu")
 		(hatch none 0.1)
-		(priority 30001)
-		(attr
-			(teardrop
-				(type padvia)
-			)
-		)
-		(connect_pads yes
-			(clearance 0)
-		)
-		(min_thickness 0.0254)
-		(fill yes
-			(island_removal_mode 1)
-		)
-		(polygon
-			(pts
-				(xy 129.336015 100.322957) (xy 129.292859 99.637014) (xy 129.031738 99.653976) (xy 128.545671 99.38403)
-				(xy 127.099081 100.011416) (xy 128.545671 100.61597) (xy 129.036638 100.341258) (xy 129.055766 100.340589)
-			)
-		)
-	)
-	(zone
-		(net "/ANT")
-		(layer "F.Cu")
-		(hatch none 0.1)
 		(priority 30000)
 		(attr
@@
 			)
 		)
+	)
+	(zone
+		(net "/ANT")
+		(layer "F.Cu")
+		(hatch none 0.1)
+		(priority 30001)
+		(attr
+			(teardrop
+				(type padvia)
+			)
+		)
+		(connect_pads yes
+			(clearance 0)
+		)
+		(min_thickness 0.0254)
+		(fill yes
+			(island_removal_mode 1)
+		)
+		(polygon
+			(pts
+				(xy 129.336015 100.322957) (xy 129.292859 99.637014) (xy 129.031738 99.653976) (xy 128.545671 99.38403)
+				(xy 127.099081 100.011416) (xy 128.545671 100.61597) (xy 129.036638 100.341258) (xy 129.055766 100.340589)
+			)
+		)
