File: ikoka-stick-meshtastic-device.kicad_sch (KiCad schematic)
At the start: 20 parts, among them J1 Conn_Coaxial, J2 Conn_01x07_Socket, J3 Conn_01x07_Socket, J4 Conn_01x02, J5 Conn_01x02, J6 Conn_01x04, Q1 AO3401A, SW1 SW_Push, U2 E22P-915M30S, U3 XIAO-ESP32-S3-SMD

Commit message: feat: v3 - swap OLED header J6 power pins (GND first), ported from tahnok fork
J6 pin 1 = GND, pin 2 = +3V3 as in tahnok 366648b; silk +/- marks.

Co-Authored-By: Claude Opus 5.5 <noreply@anthropic.com>
Claude-Session: https://claude.ai/code/session_013aihWTyEvMfq2tmgNbS7qs
Connections:
- net +3V3: now also J6.2 (Pin_2); no longer J6.1 (Pin_1)
- net GND: now also J6.1 (Pin_1); no longer J6.2 (Pin_2)
Changed lines of the file:
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@@
 	(wire
 		(pts
-			(xy 59.69 113.03) (xy 58.42 113.03)
-		)
-		(stroke
-			(width 0)
-			(type default)
-		)
-	)
-	(wire
-		(pts
 			(xy 69.85 167.64) (xy 69.85 168.91)
 		)
@@
 	(wire
 		(pts
-			(xy 58.42 109.22) (xy 58.42 110.49)
-		)
-		(stroke
-			(width 0)
-			(type default)
-		)
-	)
-	(wire
-		(pts
 			(xy 121.92 153.67) (xy 121.92 157.48)
 		)
@@
 	(wire
 		(pts
-			(xy 58.42 113.03) (xy 58.42 119.38)
-		)
-		(stroke
-			(width 0)
-			(type default)
-		)
-	)
-	(wire
-		(pts
 			(xy 63.5 69.85) (xy 74.93 69.85)
 		)
@@
 	(wire
 		(pts
-			(xy 59.69 110.49) (xy 58.42 110.49)
-		)
-		(stroke
-			(width 0)
-			(type default)
-		)
-	)
-	(wire
-		(pts
 			(xy 27.94 68.58) (xy 27.94 69.85)
 		)
@@
 	(symbol
 		(lib_id "power:GND")
-		(at 58.42 119.38 0)
-		(unit 1)
-		(body_style 1)
-		(exclude_from_sim no)
-		(in_bom yes)
-		(on_board yes)
-		(in_pos_files yes)
-		(dnp no)
-		(fields_autoplaced yes)
-		(property "Reference" "#PWR015"
-			(at 58.42 125.73 0)
-			(hide yes)
-			(show_name no)
-			(do_not_autoplace no)
-			(effects
-				(font
-					(size 1.27 1.27)
-				)
-			)
-		)
-		(property "Value" "GND"
-			(at 58.42 124.46 0)
-			(show_name no)
-			(do_not_autoplace no)
-			(effects
-				(font
-					(size 1.27 1.27)
-				)
-			)
-		)
-		(property "Footprint" ""
-			(at 58.42 119.38 0)
-			(hide yes)
-			(show_name no)
-			(do_not_autoplace no)
-			(effects
-				(font
-					(size 1.27 1.27)
-				)
-			)
-		)
-		(property "Datasheet" ""
-			(at 58.42 119.38 0)
-			(hide yes)
-			(show_name no)
-			(do_not_autoplace no)
-			(effects
-				(font
-					(size 1.27 1.27)
-				)
-			)
-		)
-		(property "Description" "Power symbol creates a global label with name \"GND\" , ground"
-			(at 58.42 119.38 0)
-			(hide yes)
-			(show_name no)
-			(do_not_autoplace no)
-			(effects
-				(font
-					(size 1.27 1.27)
-				)
-			)
-		)
-		(pin "1"
-		)
-		(instances
-			(project "ikoka-stick-meshtastic-device"
-				(path "/d817f34c-2aa5-4c70-878b-29719eb987fe"
-					(reference "#PWR015")
-					(unit 1)
-				)
-			)
-		)
-	)
-	(symbol
-		(lib_id "power:GND")
 		(at 228.6 63.5 0)
 		(unit 1)
@@
 	)
 	(symbol
-		(lib_id "power:+3V3")
-		(at 58.42 109.22 0)
-		(unit 1)
-		(body_style 1)
-		(exclude_from_sim no)
-		(in_bom yes)
-		(on_board yes)
-		(in_pos_files yes)
-		(dnp no)
-		(fields_autoplaced yes)
-		(property "Reference" "#PWR014"
-			(at 58.42 113.03 0)
-			(hide yes)
-			(show_name no)
-			(do_not_autoplace no)
-			(effects
-				(font
-					(size 1.27 1.27)
-				)
-			)
-		)
-		(property "Value" "+3V3"
-			(at 58.42 104.14 0)
-			(show_name no)
-			(do_not_autoplace no)
-			(effects
-				(font
-					(size 1.27 1.27)
-				)
-			)
-		)
-		(property "Footprint" ""
-			(at 58.42 109.22 0)
-			(hide yes)
-			(show_name no)
-			(do_not_autoplace no)
-			(effects
-				(font
-					(size 1.27 1.27)
-				)
-			)
-		)
-		(property "Datasheet" ""
-			(at 58.42 109.22 0)
-			(hide yes)
-			(show_name no)
-			(do_not_autoplace no)
-			(effects
-				(font
-					(size 1.27 1.27)
-				)
-			)
-		)
-		(property "Description" "Power symbol creates a global label with name \"+3V3\""
-			(at 58.42 109.22 0)
-			(hide yes)
-			(show_name no)
-			(do_not_autoplace no)
-			(effects
-				(font
-					(size 1.27 1.27)
-				)
-			)
-		)
-		(pin "1"
-		)
-		(instances
-			(project "ikoka-stick-meshtastic-device"
-				(path "/d817f34c-2aa5-4c70-878b-29719eb987fe"
-					(reference "#PWR014")
-					(unit 1)
-				)
-			)
-		)
-	)
-	(symbol
 		(lib_id "power:+BATT")
 		(at 240.03 107.95 0)
@@
 		)
 	)
+	(label "GND"
+		(at 59.69 110.49 180)
+		(effects
+			(font
+				(size 1.27 1.27)
+			)
+			(justify right bottom)
+		)
+	)
+	(label "+3V3"
+		(at 59.69 113.03 180)
+		(effects
+			(font
+				(size 1.27 1.27)
+			)
+			(justify right bottom)
+		)
+	)

Commit message: fix: JLCPCB PCBA rotation of pin sockets J2/J3/J6 with Fabrication Toolkit
Fabrication Toolkit ignores jlcpcb/rotations.csv; add hidden
"FT Rotation Offset" = 90 to J2, J3, J6 (positions: J2 0, J3 180, J6 90).

Co-Authored-By: Claude Opus 5.5 <noreply@anthropic.com>
Claude-Session: https://claude.ai/code/session_013aihWTyEvMfq2tmgNbS7qs
Parts:
- J2, J3, J6: FT Rotation Offset (none) -> 90
Changed lines of the file:
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@@
 			)
 		)
+    (property "FT Rotation Offset" "90" (at 143.51 165.1 0)
+      (effects (font (size 1.27 1.27)) (hide yes))
+    )
 		(pin "5"
 		)
@@
 			)
 		)
+    (property "FT Rotation Offset" "90" (at 64.77 113.03 0)
+      (effects (font (size 1.27 1.27)) (hide yes))
+    )
 		(pin "2"
 		)
@@
 			)
 		)
+    (property "FT Rotation Offset" "90" (at 46.99 165.1 0)
+      (effects (font (size 1.27 1.27)) (hide yes))
+    )
 		(pin "5"
 		)

Commit message: fix: U2 JLCPCB part to E22P-915M30S (C51912672)
U2 still carried the E22-900M30S LCSC code C411294.

Co-Authored-By: Claude Opus 5.5 <noreply@anthropic.com>
Claude-Session: https://claude.ai/code/session_013aihWTyEvMfq2tmgNbS7qs
Parts:
- U2: Check_prices https://www.snapeda.com/parts/E22-900M30S/EBYTE/view-part/?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 -> https://jlcpcb.com/partdetail/54616328-E22P915M30S/C51912672; Description_1 SX1262 868/915 MHz 1w SPI LoRa Module -> SX1262 915 MHz 1W SPI LoRa Module (E22P); LCSC C411294 -> C51912672; MP E22-900M30S -> E22P-915M30S
Changed lines of the file:
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@@
 			)
 		)
-		(property "Check_prices" "https://www.snapeda.com/parts/E22-900M30S/EBYTE/view-part/?ref=eda"
+		(property "Check_prices" "https://jlcpcb.com/partdetail/54616328-E22P915M30S/C51912672"
 			(at 205.74 46.99 0)
 			(effects
 				(font
 					(size 1.27 1.27)
-				)
-				(hide yes)
-			)
+				) (hide yes))
 		)
 		(property "STANDARD" "Manufacturer Recommendations"
@@
 			)
 		)
-		(property "MP" "E22-900M30S"
+		(property "MP" "E22P-915M30S"
 			(at 205.74 46.99 0)
 			(effects
 				(font
 					(size 1.27 1.27)
-				)
-				(hide yes)
-			)
+				) (hide yes))
 		)
-		(property "Description_1" "SX1262 868/915 MHz 1w SPI LoRa Module"
+		(property "Description_1" "SX1262 915 MHz 1W SPI LoRa Module (E22P)"
 			(at 205.74 46.99 0)
 			(effects
 				(font
 					(size 1.27 1.27)
-				)
-				(hide yes)
-			)
+				) (hide yes))
 		)
 		(property "Availability" "Not in stock"
@@
 			)
 		)
-		(property "LCSC" "C411294"
+		(property "LCSC" "C51912672"
 			(at 205.74 46.99 0)
 			(effects
 				(font
 					(size 1.27 1.27)
-				)
-				(hide yes)
-			)
+				) (hide yes))
 		)
 		(pin "1"
